File: plc esp32.kicad_pcb (KiCad board)
At the start: 2 copper layers, 155 x 122 mm, 131 parts, among them J1 Conn_01x16_Pin, J2 Conn_01x20_Pin, J3 DE9_Pins, J4 DE9_Socket, J5 RJ45_Amphenol_RJMG1BD3B8K1ANR, J7 Conn_01x03_Pin, Q1 BC547, Q2 BC547, Q3 BC547, Q4 BC547, Q5 BC547, Q6 BC547, Q7 BC547, Q8 BC547, U1 S102S01, U10 PC817, U11 PC817, U12 PC817, U13 PC817, U14 PC817, U15 PC817, U16 PC817, U17 PC817, U2 S102S01, U3 S102S01, U4 S102S01, U5 S102S01, U6 S102S01, U7 S102S01, U8 S102S01, U9 ESP32_NODEMCU

Commit message: bob
Parts:
- removed the D17 at (264.6, 49.8)
- removed the D17 at (205.6, 48.6)
- removed the D17 at (254.7, 49.8)
- removed the D17 at (244.7, 49.4)
- removed the D17 at (215.6, 49.0)
- removed the D17 at (195.7, 48.6)
- removed the D17 at (234.8, 49.4)
- removed the D17 at (225.5, 49.0)
- removed the R27 at (224.0, 63.0)
- removed the R27 at (263.1, 63.8)
- removed the R27 at (194.2, 62.6)
- removed the R27 at (243.2, 63.4)
- removed the R27 at (253.2, 63.8)
- removed the R27 at (233.3, 63.4)
- removed the R27 at (214.1, 63.0)
- removed the R27 at (204.1, 62.6)
- removed the R28 at (220.7, 60.4)
- removed the R28 at (230.6, 60.4)
- removed the R28 at (200.8, 60.0)
- removed the R28 at (210.7, 60.0)
- removed the R28 at (259.8, 61.2)
- removed the R28 at (269.7, 61.2)
- removed the R28 at (239.9, 60.8)
- removed the R28 at (249.8, 60.8)
- removed the U11 at (236.9, 53.0)
- removed the U11 at (227.6, 52.6)
- removed the U11 at (197.8, 52.2)
- removed the U11 at (217.7, 52.6)
- removed the U11 at (207.7, 52.2)
- removed the U11 at (266.7, 53.4)
- removed the U11 at (256.8, 53.4)
- removed the U11 at (246.8, 53.0)
- removed U9: ESP32_NODEMCU, imported:MODULE_ESP32_NODEMCU
- added C10: 10uF, Capacitor_THT:CP_Radial_D5.0mm_P2.50mm, F.Cu at (95.1, 71.1)
- added C11: 0.1uF, Capacitor_THT:C_Rect_L7.0mm_W2.5mm_P5.00mm, F.Cu at (101.7, 71.1)
- added C9: 1uF, Capacitor_THT:C_Disc_D5.0mm_W2.5mm_P5.00mm, F.Cu at (72.2, 54.9)
- added D17: LED, LED_THT:LED_D3.0mm, F.Cu at (122.3, 163.2)
- added J6: Conn_01x03_Pin, Connector_Phoenix_MC_HighVoltage:PhoenixContact_MC_1,5_3-G-5.08_1x03_P5.08mm_Horizontal, F.Cu at (100.2, 140.0)
- added J8: Conn_01x04_Pin, Connector_JST:JST_XH_B4B-XH-A_1x04_P2.50mm_Vertical, F.Cu at (74.9, 49.1)
- added R27: 10K, Resistor_THT:R_Axial_DIN0207_L6.3mm_D2.5mm_P7.62mm_Horizontal, F.Cu at (111.4, 162.5)
- added R28: 2.4K, Resistor_THT:R_Axial_DIN0207_L6.3mm_D2.5mm_P7.62mm_Horizontal, F.Cu at (111.4, 166.5)
- added R41: 10k, Resistor_THT:R_Axial_DIN0207_L6.3mm_D2.5mm_P7.62mm_Horizontal, F.Cu at (101.5, 212.1)
- added U11: PC817, Package_DIP:DIP-4_W7.62mm, F.Cu at (111.5, 155.8)
- added U18: ESP32-WROOM-32, RF_Module:ESP32-WROOM-32, F.Cu at (96.3, 84.1)
- J4: value DE9_Socket -> DE9_Pins; footprint Connector_Dsub:DSUB-9_Socket_Vertical_P2.77x2.84mm -> Connector_Dsub:DSUB-9_Pins_Vertical_P2.77x2.84mm
- moved R2 216.0 mm to (236.2, 99.6), turned to 180 degrees
- moved R3 211.4 mm to (234.0, 114.6), turned to 90 degrees
- moved R1 208.4 mm to (228.5, 96.2)
- moved Q1 200.9 mm to (232.6, 103.9)
- moved D2 193.5 mm to (234.4, 117.9), turned to 180 degrees
- moved D1 193.5 mm to (229.1, 118.8), turned to 90 degrees
- moved C1 191.8 mm to (229.1, 105.8), turned to 90 degrees
- moved R8 153.8 mm to (204.4, 99.6), turned to 180 degrees
- moved R9 149.9 mm to (202.2, 114.6), turned to 90 degrees
- moved R6 147.6 mm to (218.1, 114.6), turned to 90 degrees
- moved R5 147.3 mm to (220.3, 99.6), turned to 180 degrees
- moved R7 146.2 mm to (196.8, 96.2)
- moved R20 143.2 mm to (140.2, 99.6), turned to 180 degrees
- moved R4 139.9 mm to (212.7, 96.2)
- moved R21 139.2 mm to (138.0, 114.6), turned to 90 degrees
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Connections:
- J1 pad 1: unconnected-(J1-Pin_1-Pad1) -> /SSR7/SSR_B
- J1 pad 10: unconnected-(J1-Pin_10-Pad10) -> /SSR3/SSR_A
- J1 pad 11: unconnected-(J1-Pin_11-Pad11) -> /SSR2/SSR_B
- J1 pad 12: unconnected-(J1-Pin_12-Pad12) -> /SSR2/SSR_A
- J1 pad 13: unconnected-(J1-Pin_13-Pad13) -> /SSR/SSR_B
- J1 pad 14: unconnected-(J1-Pin_14-Pad14) -> /SSR/SSR_A
- J1 pad 15: unconnected-(J1-Pin_15-Pad15) -> /SSR1/SSR_B
- J1 pad 16: unconnected-(J1-Pin_16-Pad16) -> /SSR1/SSR_A
- J1 pad 2: unconnected-(J1-Pin_2-Pad2) -> /SSR7/SSR_A
- J1 pad 3: unconnected-(J1-Pin_3-Pad3) -> /SSR6/SSR_B
- J1 pad 4: unconnected-(J1-Pin_4-Pad4) -> /SSR6/SSR_A
- J1 pad 5: unconnected-(J1-Pin_5-Pad5) -> /SSR5/SSR_B
- J1 pad 6: unconnected-(J1-Pin_6-Pad6) -> /SSR5/SSR_A
- J1 pad 7: unconnected-(J1-Pin_7-Pad7) -> /SSR4/SSR_B
- J1 pad 8: unconnected-(J1-Pin_8-Pad8) -> /SSR4/SSR_A
- J1 pad 9: unconnected-(J1-Pin_9-Pad9) -> /SSR3/SSR_B
- U1 pad 1: /SSR1/SSR_A -> /SSR1/SSR_B
- U1 pad 2: /SSR1/SSR_B -> /SSR1/SSR_A
- U2 pad 1: /SSR/SSR_A -> /SSR/SSR_B
- U2 pad 2: /SSR/SSR_B -> /SSR/SSR_A
- U3 pad 1: /SSR2/SSR_A -> /SSR2/SSR_B
- U3 pad 2: /SSR2/SSR_B -> /SSR2/SSR_A
- U4 pad 1: /SSR3/SSR_A -> /SSR3/SSR_B
- U4 pad 2: /SSR3/SSR_B -> /SSR3/SSR_A
- U5 pad 1: /SSR4/SSR_A -> /SSR4/SSR_B
- U5 pad 2: /SSR4/SSR_B -> /SSR4/SSR_A
- U6 pad 1: /SSR5/SSR_A -> /SSR5/SSR_B
- U6 pad 2: /SSR5/SSR_B -> /SSR5/SSR_A
- U7 pad 1: /SSR6/SSR_A -> /SSR6/SSR_B
- U7 pad 2: /SSR6/SSR_B -> /SSR6/SSR_A
- U8 pad 1: /SSR7/SSR_A -> /SSR7/SSR_B
- U8 pad 2: /SSR7/SSR_B -> /SSR7/SSR_A
Routing:
- net GND: track 7.14 -> 151.0 mm
- net /SSR7/SSR_A: track 0.00 -> 46.7 mm
- net /SSR6/SSR_B: track 0.00 -> 39.4 mm
- net /SSR7/SSR_B: track 0.00 -> 38.9 mm
- net /SSR6/SSR_A: track 0.00 -> 37.8 mm
- net /SSR1/SSR_B: track 0.00 -> 36.7 mm
- net /SSR5/SSR_B: track 0.00 -> 32.1 mm
- net Net-(D11-K): track 0.00 -> 30.5 mm
- net Net-(D1-K): track 0.00 -> 30.5 mm
- net Net-(D10-A): track 0.00 -> 30.5 mm
- net Net-(D15-K): track 0.00 -> 30.5 mm
- net Net-(D5-K): track 0.00 -> 30.5 mm
- net Net-(D3-K): track 0.00 -> 30.5 mm
- net Net-(D13-K): track 0.00 -> 30.5 mm
- net /SSR5/SSR_A: track 0.00 -> 30.4 mm
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Other:
- board size 155 x 122 mm -> 185.8 x 122 mm
