File: plc esp32.kicad_sch (KiCad schematic)
At the start: 13 parts, among them J1 Conn_01x16_Pin, J2 Conn_01x20_Pin, J3 DE9_Pins, J4 DE9_Socket, J5 RJ45_Amphenol_RJMG1BD3B8K1ANR, J6 Conn_01x03_Pin, J7 Conn_01x03_Pin, J8 Conn_01x04_Pin, U18 ESP32-WROOM-32

Commit message: bob
Parts:
- removed J4: DE9_Socket, Connector_Dsub:DSUB-9_Socket_Vertical_P2.77x2.84mm, symbol Connector:DE9_Socket
- added J4: DE9_Pins, Connector_Dsub:DSUB-9_Pins_Vertical_P2.77x2.84mm, symbol Connector:DE9_Pins
- R41: footprint Resistor_THT:R_Axial_DIN0309_L9.0mm_D3.2mm_P12.70mm_Horizontal -> Resistor_THT:R_Axial_DIN0207_L6.3mm_D2.5mm_P7.62mm_Horizontal
Connections:
- net SSR/SIG: now also U18.23 (IO15); no longer U18.13 (IO14)
- net SSR/SSR_A: now also J1.14 (Pin_14)
- net SSR/SSR_B: now also J1.13 (Pin_13)
- net SSR1/SIG: now also U18.13 (IO14); no longer U18.23 (IO15)
- net SSR1/SSR_A: now also J1.16 (Pin_16)
- net SSR1/SSR_B: now also J1.15 (Pin_15)
- net SSR2/SSR_A: now also J1.12 (Pin_12)
- net SSR2/SSR_B: now also J1.11 (Pin_11)
- net SSR3/SSR_A: now also J1.10 (Pin_10)
- net SSR3/SSR_B: now also J1.9 (Pin_9)
- net SSR4/SSR_A: now also J1.8 (Pin_8)
- net SSR4/SSR_B: now also J1.7 (Pin_7)
- net SSR5/SSR_A: now also J1.6 (Pin_6)
- net SSR5/SSR_B: now also J1.5 (Pin_5)
- net SSR6/SSR_A: now also J1.4 (Pin_4)
- net SSR6/SSR_B: now also J1.3 (Pin_3)
- net SSR7/SSR_A: now also J1.2 (Pin_2)
- net SSR7/SSR_B: now also J1.1 (Pin_1)
Other:
- moved on the sheet: J1
