File: untitled.kicad_sch (KiCad schematic)
At the start: 8 parts, among them Q2 BC547, U2 S102S01

Commit message: bob
Parts:
- R4, R5, R6: footprint Resistor_THT:R_Axial_DIN0309_L9.0mm_D3.2mm_P12.70mm_Horizontal -> Resistor_THT:R_Axial_DIN0207_L6.3mm_D2.5mm_P7.62mm_Horizontal
Connections:
- net SSR_A: now also U2.2; no longer U2.1
- net SSR_B: now also U2.1; no longer U2.2
Changed lines of the file:
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@@
 	(hierarchical_label "SSR_B"
 		(shape input)
-		(at 181.61 105.41 0)
+		(at 181.61 100.33 0)
 		(effects
 			(font
@@
 	(hierarchical_label "SSR_A"
 		(shape input)
-		(at 181.61 100.33 0)
+		(at 181.61 105.41 0)
 		(effects
 			(font
@@
 			)
 		)
-		(property "Footprint" "Resistor_THT:R_Axial_DIN0309_L9.0mm_D3.2mm_P12.70mm_Horizontal"
+		(property "Footprint" "Resistor_THT:R_Axial_DIN0207_L6.3mm_D2.5mm_P7.62mm_Horizontal"
 			(at 140.462 114.3 90)
 			(effects
@@
 			)
 		)
-		(property "Footprint" "Resistor_THT:R_Axial_DIN0309_L9.0mm_D3.2mm_P12.70mm_Horizontal"
+		(property "Footprint" "Resistor_THT:R_Axial_DIN0207_L6.3mm_D2.5mm_P7.62mm_Horizontal"
 			(at 154.432 101.6 90)
 			(effects
@@
 			)
 		)
-		(property "Footprint" "Resistor_THT:R_Axial_DIN0309_L9.0mm_D3.2mm_P12.70mm_Horizontal"
+		(property "Footprint" "Resistor_THT:R_Axial_DIN0207_L6.3mm_D2.5mm_P7.62mm_Horizontal"
 			(at 134.62 112.268 90)
 			(effects
